File: alto_driver.kicad_pcb (KiCad board)
At the start: 2 copper layers, 73 parts, among them IC1 AS5047P-ATSM, J1 Conn_01x04_Pin, J2 Conn_01x02_Pin, J3 XT30PW_2_2_-M.G.B, J4 XT30PW_2_2_-M.G.B, J5 Conn_01x04_Pin, J6 Conn_01x02_Pin, U1 LMR33620ADDA, U2 TLV75533PDBVR, U3 STM32G431CBT6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

Commit message: 0314
Parts:
- added H1: MountingHole, MountingHole:MountingHole_3.2mm_M3, F.Cu at (165.5, 84.5)
- added H2: MountingHole, MountingHole:MountingHole_3.2mm_M3, F.Cu at (134.5, 115.5)
- C28, C30, C31, C33, R11, R14, R15, R16, U6: moved to B.Cu
- U7: renamed from IC1; moved to B.Cu
- moved J3 81.7 mm to (174.0, 100.0), turned to 90 degrees
- moved J1 73.5 mm to (161.9, 119.2), turned to -90 degrees
- moved C26 65.8 mm to (157.4, 115.3), turned to -90 degrees
- moved C25 65.0 mm to (147.6, 117.9), turned to 180 degrees
- moved U4 64.3 mm to (161.9, 113.9), turned to 180 degrees
- moved C10 61.3 mm to (168.7, 89.9), turned to 90 degrees
- moved C9 60.6 mm to (167.2, 89.9), turned to 90 degrees
- moved C8 60.1 mm to (165.7, 89.9), turned to 90 degrees
- moved R12 59.6 mm to (154.6, 112.3)
- moved D3 59.1 mm to (139.8, 119.1), turned to 180 degrees
- moved C20 58.2 mm to (150.5, 117.9), turned to 180 degrees
- moved U7 56.7 mm to (150.0, 100.0)
- moved C16 56.2 mm to (141.1, 111.8), turned to -90 degrees
- moved C15 55.8 mm to (141.1, 108.8), turned to 90 degrees
- moved C19 55.4 mm to (153.5, 108.9), turned to -90 degrees
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Connections:
- J1 pad 1: SWDIO -> +3.3V
- J1 pad 2: SWCLK -> GND
- J1 pad 3: GND -> SWDIO
- J1 pad 4: +3.3V -> SWCLK
- J3 pad N: +24V -> GND
- J3 pad P: GND -> +24V
- J4 pad N: +24V -> GND
- J4 pad P: GND -> +24V
- J5 pad 1: A1 -> B2
- J5 pad 2: A2 -> B1
- J5 pad 3: B1 -> A1
- J5 pad 4: B2 -> A2
- R10 pad 1: SCK -> SPI2_SCK
- R11 pad 1: MISO -> SPI2_MISO
- R12 pad 1: MOSI -> SPI2_MOSI
- R13 pad 1: USART2_TX -> USART1_TX
- R13 pad 2: USART2_RX -> USART1_RX
- R17 pad 2: Net-(U3-PB3) -> Net-(U3-PA4)
- R19 pad 2: Net-(U3-PB4) -> Net-(U3-PA3)
- R6 pad 2: SDA -> I2C2_SDA
- R7 pad 2: SCL -> I2C2_SCL
- R9 pad 1: CS -> SPI2_CS
- U3 pad 10: USART2_TX -> unconnected-(U3-PA2-Pad10)
- U3 pad 11: USART2_RX -> Net-(U3-PA3)
- U3 pad 12: EN -> Net-(U3-PA4)
- U3 pad 13: SPI1_SCK -> unconnected-(U3-PA5-Pad13)
- U3 pad 14: SPI1_MISO -> unconnected-(U3-PA6-Pad14)
- U3 pad 15: SPI1_MOSI -> unconnected-(U3-PA7-Pad15)
- U3 pad 16: SPI1_CS -> unconnected-(U3-PB0-Pad16)
- U3 pad 2: DIAG -> unconnected-(U3-PC13-Pad2)
- U3 pad 25: unconnected-(U3-PB11-Pad25) -> LIMIT_SW
- U3 pad 26: unconnected-(U3-PB12-Pad26) -> SPI2_CS
- U3 pad 27: unconnected-(U3-PB13-Pad27) -> SPI2_SCK
- U3 pad 28: unconnected-(U3-PB14-Pad28) -> SPI2_MISO
- U3 pad 29: unconnected-(U3-PB15-Pad29) -> SPI2_MOSI
- U3 pad 30: unconnected-(U3-PA8-Pad30) -> I2C2_SDA
- U3 pad 31: unconnected-(U3-PA9-Pad31) -> I2C2_SCL
- U3 pad 39: I2C1_SCL -> EN
- U3 pad 40: Net-(U3-PB3) -> DIR
- U3 pad 41: Net-(U3-PB4) -> STEP
- U3 pad 42: unconnected-(U3-PB5-Pad42) -> DIAG
- U3 pad 43: unconnected-(U3-PB6-Pad43) -> USART1_TX
- U3 pad 44: I2C1_SDA -> USART1_RX
- U3 pad 46: LIMIT_SW -> unconnected-(U3-PB9-Pad46)
- U3 pad 8: STEP -> unconnected-(U3-PA0-Pad8)
- U3 pad 9: DIR -> unconnected-(U3-PA1-Pad9)
- U4 pad 5: SDA -> I2C2_SDA
- U4 pad 6: SCL -> I2C2_SCL
- U6 pad 14: USART2_RX -> USART1_RX
Routing:
- net +3.3V: track 0.00 -> 152.3 mm, vias 0 -> 8
- net GND: track 0.00 -> 147.1 mm, vias 0 -> 28
- net +24V: track 0.00 -> 135.9 mm, vias 0 -> 6
- net CANH: track 0.00 -> 57.4 mm
- net DIR: track 0.00 -> 52.2 mm, vias 0 -> 1
- net CANL: track 0.00 -> 50.7 mm, vias 0 -> 3
- net STEP: track 0.00 -> 42.3 mm, vias 0 -> 3
- net USART1_RX: track 0.00 -> 41.1 mm, vias 0 -> 3
- net EN: track 0.00 -> 36.7 mm, vias 0 -> 1
- net DIAG: track 0.00 -> 25.2 mm, vias 0 -> 3
- net Net-(U6-BRA): track 0.00 -> 24.3 mm, vias 0 -> 2
- net +5V: track 0.00 -> 24.1 mm
- net FDCAN1_RX: track 0.00 -> 23.5 mm, vias 0 -> 2
- net Net-(U6-BRB): track 0.00 -> 22.8 mm, vias 0 -> 2
- net LIMIT_SW: track 0.00 -> 20.8 mm
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- added copper zone on In1.Cu, net GND
Other:
- board outline added: 42 x 42 mm
- copper layers 2 -> 4
- rule pad_to_mask_clearance: 0 -> 0.1

Commit message: 0321
Parts:
- C29, C32: moved to B.Cu
- moved C32 35.2 mm to (111.5, 100.5)
- moved C29 35.2 mm to (114.7, 100.5), turned to -90 degrees
- moved C6 9.71 mm to (137.0, 94.2), turned to -90 degrees
- moved U1 9.70 mm to (143.8, 95.7)
- moved C27 8.92 mm to (162.5, 100.7)
- moved D2 8.92 mm to (152.0, 100.6)
- moved U5 8.92 mm to (157.8, 100.6)
- moved C2 8.25 mm to (138.0, 90.0), turned to -90 degrees
- moved C5 7.37 mm to (138.8, 94.2), turned to -90 degrees
- moved D1 6.31 mm to (143.7, 90.0)
- moved C1 6.17 mm to (134.5, 90.0), turned to -90 degrees
- moved C7 6.04 mm to (149.8, 88.5)
- moved C12 5.81 mm to (149.8, 91.5)
- moved R1 5.81 mm to (149.8, 93.0)
- moved R2 5.81 mm to (149.8, 94.5)
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Routing:
- net +3.3V: track 152.3 -> 0.00 mm, vias 8 -> 0
- net GND: track 147.1 -> 0.00 mm, vias 28 -> 0
- net +24V: track 135.9 -> 0.00 mm, vias 6 -> 0
- net CANH: track 57.4 -> 0.00 mm
- net DIR: track 52.2 -> 0.00 mm, vias 1 -> 0
- net CANL: track 50.7 -> 0.00 mm, vias 3 -> 0
- net STEP: track 42.3 -> 0.00 mm, vias 3 -> 0
- net USART1_RX: track 41.1 -> 0.00 mm, vias 3 -> 0
- net EN: track 36.7 -> 0.00 mm, vias 1 -> 0
- net DIAG: track 25.2 -> 0.00 mm, vias 3 -> 0
- net Net-(U6-BRA): track 24.3 -> 0.00 mm, vias 2 -> 0
- net +5V: track 24.1 -> 0.00 mm
- net FDCAN1_RX: track 23.5 -> 0.00 mm, vias 2 -> 0
- net Net-(U6-BRB): track 22.8 -> 0.00 mm, vias 2 -> 0
- net LIMIT_SW: track 20.8 -> 0.00 mm
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Other:
- board size 42 x 42 mm -> 40 x 35 mm
