File: alto_driver.kicad_sch (KiCad schematic)
At the start: 26 parts, among them IC1 AS5047P-ATSM, U1 LMR33620ADDA, U2 TLV75533PDBVR, U3 STM32G431CBTx, U4 AT24C32D-SSHM-B, U5 TCAN3413DR, U6 TMC2209-LA

Commit message: v1
Parts:
- added C15, C16: 30pF/10V, symbol Device:C
- added C17, C18, C19, C20, C21, C25, C26, C27, C28: 100nF/10V, symbol Device:C
- added C22: 10uF/10V, symbol Device:C
- added C23, C24: 1uF/10V, symbol Device:C
- added C29, C33: 100nF/50V, symbol Device:C
- added C30: 22nF/50V, symbol Device:C
- added C31: 2.2uF/50V, symbol Device:C
- added C32: 100uF/50V, symbol Device:C
- added D2: PESD2CAN, PESD2CAN:SOT95P230X110-3N, symbol PESD2CAN:PESD2CAN
- added D3: LED/BLUE, symbol Device:LED
- added D4: LED/GREEN, symbol Device:LED
- added D5: LED/RED, symbol Device:LED
- added FB1: FerriteBead, symbol Device:FerriteBead
- added J1, J3, J4, J5: Conn_01x04_Pin, symbol Connector:Conn_01x04_Pin
- added J2: Conn_01x02_Pin, symbol Connector:Conn_01x02_Pin
- added R10, R11, R12, R9: 33R, symbol Device:R
- added R13: 1kR, symbol Device:R
- added R14, R15: 0.12R, symbol Device:R
- added R16, R4, R5: 10kR, symbol Device:R
- added R17, R18, R19: 1KR, symbol Device:R
- added R6, R7: 4.7kR, symbol Device:R
- added R8: 120R, symbol Device:R
- added Y1: 16MHz/20pF, symbol Device:Crystal_GND24
- U3: value STM32G431CBTx -> STM32G431CBT6
Connections:
- net +24V: now also U6.22 (VS), U6.28 (VS), C29.1, C32.1, J3.4 (Pin_4), J4.4 (Pin_4)
- net +3.3V: now also IC1.11 (VDD), IC1.12 (VDD3V), U3.1 (VBAT), U3.24 (VDD), U3.36 (VDD), U3.48 (VDD), U4.8 (VCC), U5.3 (VCC), U5.5 (SHDNV_IO), U6.15 (VCC_IO), C18.1, C19.1, C20.1, C21.1, C22.1, C23.1, C26.2, C27.2, C28.2, FB1.2, J1.4 (Pin_4), R16.2, R18.2, R4.1, R6.1, R7.1
- net AGND: now also IC1.13 (GND), U3.19 (VSSA), U3.23 (VSS), U3.35 (VSS), U3.47 (VSS), U4.1 (A0), U4.2 (A1), U4.3 (A2), U4.4 (GND), U4.7 (WP), U5.2 (GND), U5.8 (STB), U6.10 (MS2/AD1), U6.13 (CLK), U6.18 (GND), U6.20 (STDBY), U6.29 (GND), U6.3 (GND), U6.7 (SPREAD), U6.9 (MS1/AD0), C15.2, C16.2, C17.2, C18.2, C19.2, C20.2, C21.2, C22.2, C23.2, C24.2, C25.2, C26.1, C27.1, C28.1, C31.2, C32.2, C33.2, D2.3, D3.1 (K), D4.1 (K), D5.1 (K), J1.3 (Pin_3), J3.3 (Pin_3), J4.3 (Pin_3), R14.2, R15.2, R5.1, Y1.2 (G), Y1.4 (G)
- net SDA: now reaches U4.5 (SDA)
- net SDA: now also R6.2
- net SCL: now reaches U4.6 (SCL)
- net SCL: now also R7.2
- net USART2_TX: now reaches U3.10 (PA2)
- net USART2_TX: now also R13.1
- net USART2_RX: now reaches U3.11 (PA3)
- net USART2_RX: now also U6.14 (~{PD}/UART), R13.2
- net EN: now reaches U3.12 (PA4)
- net EN: now also U6.2 (~{EN})
- net SPI1_SCK: now reaches U3.13 (PA5)
- net SPI1_MISO: now reaches U3.14 (PA6)
- net SPI1_MOSI: now reaches U3.15 (PA7)
- net SPI1_CS: now reaches U3.16 (PB0)
- net DIAG: now reaches U3.2 (PC13)
- net DIAG: now also U6.11 (DIAG)
- net +3.3VA: now reaches U3.20 (VREF+)
- net +3.3VA: now also U3.21 (VDDA), C24.1, C25.1, FB1.1
- net FDCAN1_RX: now reaches U3.33 (PA11)
- net FDCAN1_RX: now also U5.4 (RXD)
- net FDCAN1_TX: now reaches U3.34 (PA12)
- net FDCAN1_TX: now also U5.1 (TXD)
- net SWDIO: now reaches U3.37 (PA13)
- net SWDIO: now also J1.1 (Pin_1)
- net SWCLK: now reaches U3.38 (PA14)
- net SWCLK: now also J1.2 (Pin_2)
- net I2C1_SCL: now reaches U3.39 (PA15)
- net at U3.40 (PB3): now also R17.2
- net at U3.41 (PB4): now also R19.2
- net I2C1_SDA: now reaches U3.44 (PB7)
- net at U3.45 (PB8): now also R5.2
- net OSC_IN: now reaches U3.5 (PF0)
- net OSC_IN: now also C15.1, Y1.1
- net OSC_OUT: now reaches U3.6 (PF1)
- net OSC_OUT: now also C16.1, Y1.3
- net at U3.7 (PG10): now also C17.1, R4.2
- net STEP: now reaches U3.8 (PA0)
- net STEP: now also U6.16 (STEP)
- net DIR: now reaches U3.9 (PA1)
- net DIR: now also U6.19 (DIR)
- net B2: now reaches U6.1 (OB2)
- net B2: now also J5.4 (Pin_4)
- net at U6.17 (VREF): now also C33.1, R16.1
- net A2: now reaches U6.21 (OA2)
- net A2: now also J5.2 (Pin_2)
- net at U6.23 (BRA): now also R14.1
- net A1: now reaches U6.24 (OA1)
- net A1: now also J5.1 (Pin_1)
- net B1: now reaches U6.26 (OB1)
- net B1: now also J5.3 (Pin_3)
- net at U6.27 (BRB): now also R15.1
- net at U6.4 (CPO): now also C30.1
- net at U6.5 (CPI): now also C30.2
- net at U6.6 (VCP): now also C29.2
- net at U6.8 (5VOUT): now also C31.1
- net CANL: now reaches U5.6 (CANL)
- net CANL: now also D2.2, J3.2 (Pin_2), J4.2 (Pin_2), R8.2
- net CANH: now reaches U5.7 (CANH)
- net CANH: now also D2.1, J2.2 (Pin_2), J3.1 (Pin_1), J4.1 (Pin_1)
- net at IC1.1 (CSN): now also R9.2
- net at IC1.2 (CLK): now also R10.2
- net at IC1.3 (MISO): now also R11.2
- net at IC1.4 (MOSI): now also R12.2
- new net: J2.1 (Pin_1), R8.1
- new net: D3.2 (A), R17.1
- new net: D5.2 (A), R19.1
- new net: D4.2 (A), R18.1
- new net CS: R9.1
- new net MISO: R11.1
- new net MOSI: R12.1
- new net SCK: R10.1
- no-connect marks 0 -> 9
Other:
- note added: "24V power input protection"
- note added: "24V to 5V DC-DC converter"
- note added: "5V to 3.3V LDO converter"
- note added: "Connector"
- note added: "EEPROM"
- note added: "FD CAN transceiver"
- note added: "Magnet angle sensor"
- note added: "STM32 controller unit"
- note added: "Stepper driver"
- moved on the sheet: C1, C10, C11, C12, C13, C14, C2, C3, C4, C5, C6, C7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

Commit message: 0309
Parts:
- removed J3, J4: Conn_01x04_Pin, symbol Connector:Conn_01x04_Pin
- added J3, J4: XT30PW_2_2_-M.G.B, XT30PW_2_2_-M.G.B:AMASS_XT30PW_2_2_-M.G.B, symbol XT30PW_2_2_-M.G.B:XT30PW_2_2_-M.G.B
- added J6: Conn_01x02_Pin, Connector_JST:JST_XH_S2B-XH-A_1x02_P2.50mm_Horizontal, symbol Connector:Conn_01x02_Pin
- C1, C2, C3, C32, C4: footprint (none) -> Capacitor_SMD:C_1210_3225Metric
- C10, C11, C12, C13, C14, C15, C16, C17, C18, C19, C20, C21, C22, C23, C24, C25, C26, C27, C28, C29, C30, C31, C33, C5, C6, C7, C8, C9: footprint (none) -> Capacitor_SMD:C_0603_1608Metric
- D1: footprint (none) -> Diode_SMD:D_SMB
- D3, D4, D5: footprint (none) -> LED_SMD:LED_0603_1608Metric
- FB1: footprint (none) -> Inductor_SMD:L_0603_1608Metric
- IC1: footprint SOP65P640X120-14N -> AS5047P-ATSM:SOP65P640X120-14N
- J1: footprint (none) -> Connector_PinHeader_2.54mm:PinHeader_1x04_P2.54mm_Vertical
- J2: footprint (none) -> Connector_PinHeader_2.54mm:PinHeader_1x02_P2.54mm_Vertical
- J5: footprint (none) -> Connector_JST:JST_XH_S4B-XH-A_1x04_P2.50mm_Horizontal
- L1: footprint (none) -> Inductor_SMD:L_Chilisin_BWVS00505030
- R1: value 24.9kR -> 24.9KR; footprint (none) -> Resistor_SMD:R_0603_1608Metric
- R10, R11, R12, R17, R18, R19, R8, R9: footprint (none) -> Resistor_SMD:R_0603_1608Metric
- R13: value 1kR -> 1KR; footprint (none) -> Resistor_SMD:R_0603_1608Metric
- R14, R15: footprint (none) -> Resistor_SMD:R_1206_3216Metric
- R16, R4, R5: value 10kR -> 10KR; footprint (none) -> Resistor_SMD:R_0603_1608Metric
- R2, R3: value 100kR -> 100KR; footprint (none) -> Resistor_SMD:R_0603_1608Metric
- R6, R7: value 4.7kR -> 4.7KR; footprint (none) -> Resistor_SMD:R_0603_1608Metric
- U4: footprint SOIC127P600X175-8N -> AT24C32D-SSHM-T:SOIC127P600X175-8N
- U5: footprint SOIC127P600X175-8N -> TCAN3413DR:SOIC127P600X175-8N
- U6: footprint Package_DFN_QFN:VQFN-28-1EP_5x5mm_P0.5mm_EP3.7x3.7mm_ThermalVias -> TMC2209-LA:QFN50P500X500X90-29N
- Y1: footprint (none) -> Crystal:Crystal_SMD_3225-4Pin_3.2x2.5mm
Connections:
- net +24V: now also J3.N, J4.N
- net AGND: now also J3.P, J4.P, J6.2 (Pin_2)
- net CANH: now also J3.S1, J4.S1
- net CANL: now also J3.S2, J4.S2
- net LIMIT_SW: now reaches U3.46 (PB9)
- net LIMIT_SW: now also J6.1 (Pin_1)
Other:
- moved on the sheet: J1, R5

Commit message: 0314
Parts:
- added H1, H2: MountingHole, MountingHole:MountingHole_3.2mm_M3, symbol Mechanical:MountingHole
- renumbered IC1 to U7
Connections:
- net CS is gone; now on net SPI2_CS: R9.1
- net I2C1_SCL is gone; now on net EN: U3.39 (PA15)
- net MISO is gone; now on net SPI2_MISO: R11.1
- net MOSI is gone; now on net SPI2_MOSI: R12.1
- net SCK is gone; now on net SPI2_SCK: R10.1
- net SCL is gone; now on net I2C2_SCL: R7.2, U4.6 (SCL)
- net SDA is gone; now on net I2C2_SDA: R6.2, U4.5 (SDA)
- net +24V: now also J3.P, J4.P; no longer J3.N, J4.N
- net +3.3V: now also J1.1 (Pin_1); no longer J1.4 (Pin_4)
- net A1: now also J5.3 (Pin_3); no longer J5.1 (Pin_1)
- net A2: now also J5.4 (Pin_4); no longer J5.2 (Pin_2)
- net AGND: now also J1.2 (Pin_2), J3.N, J4.N; no longer J1.3 (Pin_3), J3.P, J4.P
- net B1: now also J5.2 (Pin_2); no longer J5.3 (Pin_3)
- net B2: now also J5.1 (Pin_1); no longer J5.4 (Pin_4)
- net DIAG: now also U3.42 (PB5); no longer U3.2 (PC13)
- net DIR: now also U3.40 (PB3); no longer U3.9 (PA1)
- net EN: no longer U3.12 (PA4)
- net LIMIT_SW: now also U3.25 (PB11); no longer U3.46 (PB9)
- net STEP: now also U3.41 (PB4); no longer U3.8 (PA0)
- net SWCLK: now also J1.4 (Pin_4); no longer J1.2 (Pin_2)
- net SWDIO: now also J1.3 (Pin_3); no longer J1.1 (Pin_1)
- net SPI2_CS: now reaches U3.26 (PB12)
- net SPI2_SCK: now reaches U3.27 (PB13)
- net SPI2_MISO: now reaches U3.28 (PB14)
- net SPI2_MOSI: now reaches U3.29 (PB15)
- net I2C2_SDA: now reaches U3.30 (PA8)
- net I2C2_SCL: now reaches U3.31 (PA9)
- net at R17.2: now also U3.12 (PA4); no longer U3.40 (PB3)
- net at R19.2: now also U3.11 (PA3); no longer U3.41 (PB4)
- net USART1_TX: now reaches U3.43 (PB6)
- net USART1_TX: now also R13.1
- net I2C1_SDA renamed USART1_RX
- net USART1_RX: now also R13.2, U6.14 (~{PD}/UART)
- net SPI1_CS: no longer names the net of U3.16 (PB0)
- net SPI1_MISO: no longer names the net of U3.14 (PA6)
- net SPI1_MOSI: no longer names the net of U3.15 (PA7)
- net SPI1_SCK: no longer names the net of U3.13 (PA5)
- removed net USART2_RX: R13.2, U3.11 (PA3), U6.14 (~{PD}/UART)
- net USART2_TX: no longer names the net of U3.10 (PA2)
- net USART2_TX: no longer R13.1
- no-connect marks 9 -> 25
Other:
- moved on the sheet: D3, D5, R17, R19, R5, R7

Commit message: 0321
Parts:
- FB1: value FerriteBead -> 600R/25%
Changed lines of the file:
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@@
 			)
 		)
-		(property "Value" "FerriteBead"
+		(property "Value" "600R/25%"
 			(at 377.1392 40.64 90)
 			(effects
