File: alto_driver_42.kicad_pcb (KiCad board)
At the start: 4 copper layers, 42 x 42 mm, 75 parts, among them J1 Conn_01x04_Pin, J2 Conn_01x02_Pin, J3 XT30PW_2_2_-M.G.B, J4 XT30PW_2_2_-M.G.B, J5 Conn_01x04_Pin, J6 Conn_01x02_Pin, U1 LMR33620ADDA, U2 TLV75533PDBVR, U3 STM32G431CBT6, U4 AT24C32D-SSHM-B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

Commit message: 0321
Parts:
- C29, C32: moved to B.Cu
- moved C32 4.06 mm to (150.0, 93.2), turned to 0 degrees
- moved C29 3.31 mm to (145.8, 93.3)
Routing:
- net Net-(U6-VCP): track 9.89 -> 2.87 mm, vias 1 -> 0
- net +24V: track 135.9 -> 130.5 mm
- net GND: track 147.1 -> 142.0 mm, vias 28 -> 31
- net +3.3V: track 152.3 -> 156.3 mm
- net DIR: track 52.2 -> 49.8 mm
- net SWDIO: track 17.6 -> 16.6 mm
- net EN: track 36.7 -> 37.6 mm
- net PG: track 12.8 -> 13.6 mm
